File: Schema/Keypad/Keypad.kicad_pcb (KiCad board)
At the start: 2 copper layers, 76.8 x 117.6 mm, 75 parts, among them J1 JSTBATT, J2 Conn_01x04_Socket, J3 Conn_01x03_Socket, Q1 2N7002, Q2 AO3401A, Q4 2N7002, SW1 SW_SPDT, U1 BQ24075RGT, U2 nRF52840_holyiot_18010, U3 XC6206PxxxMR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

Commit message: Updating with enclosure
Parts:
- moved D16 17.9 mm to (119.0, 159.5)
- renumbered Q4 to Q3, R16 to R13, R13 to R15, R15 to R16
Routing:
- net ROW4: track 134.8 -> 150.9 mm, vias 0 -> 4
- net Net-(D16-A): track 4.11 -> 16.1 mm, vias 0 -> 1
Other:
- outline, holes or cut-outs redrawn
